File: balun_amp.kicad_pcb (KiCad board)
At the start: 2 copper layers, 44 parts, among them J1 Input, J2 Output, J3 USB_B_Micro, U1 LT1226, U2 LT1226, U3 LT1226, U4 BQ2404x, U5 NMA0512SC, U6 TPS61027

Commit message: no change
Parts:
- added C12: 1u, Capacitor_SMD:C_0603_1608Metric_Pad1.05x0.95mm_HandSolder, F.Cu at (53.7, 12.2)
- added C13: 1u, Capacitor_SMD:C_0603_1608Metric_Pad1.05x0.95mm_HandSolder, F.Cu at (53.7, 14.7)
- added C14: 10n, Capacitor_SMD:C_0402_1005Metric, F.Cu at (57.4, 11.9)
- added C15: 10n, Capacitor_SMD:C_0402_1005Metric, F.Cu at (53.0, 16.9)
- added C16: 10n, Capacitor_SMD:C_0402_1005Metric, F.Cu at (57.4, 13.9)
- added C17: 10n, Capacitor_SMD:C_0402_1005Metric, F.Cu at (60.3, 11.9)
- added C18: 10n, Capacitor_SMD:C_0402_1005Metric, F.Cu at (55.9, 16.9)
- added C19: 10n, Capacitor_SMD:C_0402_1005Metric, F.Cu at (60.3, 13.9)
- added C20: 10n, Capacitor_SMD:C_0402_1005Metric, F.Cu at (58.8, 15.9)
- C1, C2, C5, C6: value C -> 10u
- C10: value C -> 100n
- C7, C8, C9: value C -> 1u
- L2, L3: value L -> 150u
Other:
- copper layers 2 -> 4

Commit message: Layout update
Parts:
- moved C20 98.3 mm to (109.2, 100.3), turned to 270 degrees
- moved C19 93.8 mm to (109.2, 94.0), turned to 270 degrees
- moved C12 91.7 mm to (113.0, 82.2), turned to 90 degrees
- moved C17 86.7 mm to (110.5, 82.5), turned to 90 degrees
- moved C15 86.1 mm to (100.3, 88.9), turned to 270 degrees
- moved C13 76.3 mm to (110.5, 65.6), turned to 90 degrees
- moved C14 73.1 mm to (100.3, 71.1), turned to 270 degrees
- moved C18 71.5 mm to (108.0, 66.0), turned to 90 degrees
- moved C16 60.1 mm to (100.3, 55.9), turned to 270 degrees
- moved C4 56.9 mm to (133.3, 48.3), turned to 270 degrees
- moved J2 53.5 mm to (144.8, 74.9)
- moved L1 48.1 mm to (142.2, 57.1), turned to 90 degrees
- moved R9 43.1 mm to (112.5, 55.9)
- moved R7 43.0 mm to (83.8, 78.7), turned to 180 degrees
- moved U1 41.9 mm to (98.4, 64.8), turned to 90 degrees
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Connections:
- net Net-(J1-Pad1) renamed /input+
- net Net-(J1-Pad2) renamed /input-
Routing:
- net /input-: track 0.00 -> 1.79 mm
- net /input+: track 0.00 -> 1.79 mm
- added copper zone on F.Cu, net GND
