File: balun_amp.sch (KiCad schematic (older format))
At the start: 12 parts

Commit message: add 5v to +/-12V, add battery charger
Parts:
- added BT?: Battery_Cell, symbol Device:Battery_Cell
- added C? (x4): C, symbol Device:C
- added D? (x2): LED, symbol Device:LED
- added J?: USB_B_Micro, symbol Connector:USB_B_Micro
- added L? (x2): L, symbol Device:L
- added R?: 2k, symbol Device:R
- added R?: 1k, symbol Device:R
- added R? (x2): 1.5k, symbol Device:R
- added R?: 10k, symbol Device:R
- added U?: NMA0512SC, Converter_DCDC:Converter_DCDC_muRata_NMAxxxxSC_THT, symbol Regulator_Switching:NMA0512SC
- added U?: BQ2404x, symbol balun_amp:BQ2404x
- U? (x3): symbol diff_amp:LT1226 -> balun_amp:LT1226
- gave numbers to parts that had none: 9
Connections:
- net labels added: +5V, +BATT, -BATT, GNDPWR, INN, INP, VBUS, Vout
- wire segments 29 -> 85

Commit message: add 5v boost converter
Parts:
- added C?: 10u, symbol Device:C
- added C?: 2.2u, symbol Device:C
- added C?: 47u, symbol Device:C
- added D?: LED, symbol Device:LED
- added L?: 6.8uH, symbol Device:L
- added R?: 8.5k, symbol Device:R
- added R? (x2): 1.5k, symbol Device:R
- added U?: TPS61027, symbol balun_amp:TPS6102x
Connections:
- wire segments 85 -> 115

Commit message: finish the draft schematic, generate the netlist and assign the footprint
Parts:
- added C10: C, Capacitor_SMD:C_0402_1005Metric, symbol Device:C
- added C7, C8, C9: C, Capacitor_SMD:C_0603_1608Metric_Pad1.05x0.95mm_HandSolder, symbol Device:C
- added J1: Input, Connector_Coaxial:SMA_Amphenol_132289_EdgeMount, symbol Connector:Conn_Coaxial
- added J2: Output, Connector_Coaxial:SMA_Amphenol_132289_EdgeMount, symbol Connector:Conn_Coaxial
- BT1: renamed from BT?; footprint (none) -> Battery:BatteryHolder_MPD_BH-18650-PC2
- C1, C2, C3, C4, C5, C6: renamed from C?; footprint (none) -> Capacitor_SMD:C_0603_1608Metric_Pad1.05x0.95mm_HandSolder
- C11: renamed from C?; footprint (none) -> Capacitor_SMD:C_0805_2012Metric_Pad1.15x1.40mm_HandSolder
- D1, D2, D3: renamed from D?; footprint (none) -> LED_SMD:LED_0603_1608Metric_Pad1.05x0.95mm_HandSolder
- J3: renamed from J?; footprint (none) -> Connector_USB:USB_Micro-B_Molex_47346-0001
- L1: renamed from L?; footprint (none) -> Inductor_SMD:L_Coilcraft_XAL5030
- L2, L3: renamed from L?; footprint (none) -> Inductor_SMD:L_0805_2012Metric_Pad1.15x1.40mm_HandSolder
- R1, R2, R3, R4, R5, R6, R7, R8: footprint (none) -> Resistor_SMD:R_0402_1005Metric
- R10, R9: renamed from R?; footprint (none) -> Resistor_SMD:R_0402_1005Metric
- R11, R12, R13, R14, R15, R16: renamed from R?; footprint (none) -> Resistor_SMD:R_0603_1608Metric_Pad1.05x0.95mm_HandSolder
- Rg1: renamed from Rg; footprint (none) -> Resistor_SMD:R_0402_1005Metric
- U1, U2, U3: renamed from U?; footprint (none) -> Package_SO:SOIC-8_3.9x4.9mm_P1.27mm
- U4: renamed from U?; footprint (none) -> Package_SON:WSON-10-1EP_2x3mm_P0.5mm_EP0.84x2.4mm
- U6: renamed from U?; footprint (none) -> Package_SON:VSON-10-1EP_3x3mm_P0.5mm_EP1.65x2.4mm_ThermalVias
- gave numbers to parts that had none: 1
Connections:
- net labels removed: INN, INP, Vout
- wire segments 115 -> 129

Commit message: Update capacitor value and package
Parts:
- added C12, C13: 1u, Capacitor_SMD:C_0603_1608Metric_Pad1.05x0.95mm_HandSolder, symbol Device:C
- added C14, C15, C16, C17, C18, C19, C20: 10n, Capacitor_SMD:C_0402_1005Metric, symbol Device:C
- C1, C2, C5, C6: value C -> 10u
- C10: value C -> 100n
- C7, C8, C9: value C -> 1u
- L2, L3: value L -> 150u
Connections:
- wire segments 129 -> 149
Other:
- note added: "Pin 1 & 8 are left for null balancing, \nneed additional tuning if the opamp is not balance."
- note added: "Use 18650 battery"
- note added: "VDD=+12V\nVSS=-12V"

Commit message: Layout update
Parts:
- BT1: symbol Device:Battery_Cell -> balun_amp-rescue:Battery_Cell-Device
- C1, C10, C11, C12, C13, C14, C15, C16, C17, C18, C19, C2, C20, C3, C4, C5, C6, C7, C8, C9: symbol Device:C -> balun_amp-rescue:C-Device
- D1, D2, D3: symbol Device:LED -> balun_amp-rescue:LED-Device
- J1, J2: symbol Connector:Conn_Coaxial -> balun_amp-rescue:Conn_Coaxial-Connector
- J3: symbol Connector:USB_B_Micro -> balun_amp-rescue:USB_B_Micro-Connector
- L1, L2, L3: symbol Device:L -> balun_amp-rescue:L-Device
- R1, R10, R11, R12, R13, R14, R15, R16, R2, R3, R4, R5, R6, R7, R8, R9, Rg1: symbol Device:R -> balun_amp-rescue:R-Device
- U5: symbol Regulator_Switching:NMA0512SC -> balun_amp-rescue:NMA0512SC-Regulator_Switching
Connections:
- net labels added: input+, input-
